File: SmartNode/eagle/main-01.brd (EAGLE design)
At the start: 131.8 x 67 mm, 151 parts, among them IC1 ATmega328P-AU, IC2 MAX3468CSA, IC4 78L33, IC5 MCP23017-E/SO-SOIC28, IC6 TPS56X200, IC7 LTC1694, Q1 IRLML2502, X0 OPI-ZERO

Commit message: Ann component values to schematic
Parts:
- R15, R16, R18, R19, R21, R24, R26, R27, R32, R36, R39, R43, R44, R46, R47: value (none) -> 390
- R17, R20, R25, R31, R37, R42, R45, R48: value (none) -> 51
- R49, R50, R51, R52, R53, R54, R55, R56, R57, R58, R59, R60, R61, R62, R63, R64, R66: value (none) -> 10K
- R6, R7: value 4.7K -> NI
- R65: value (none) -> 750
- R9: value (none) -> 120
