File: SmartNode/eagle/main-stm-03.1.sch (EAGLE design)
At the start: 152 parts, among them IC2 MAX3468CSA, IC4 78L33, IC5 MCP23017-E/SO-SOIC28, IC6 TPS56X200, IC7 LTC1694, Q1 IRLML2502, Q2 IRLML2502, U2 STM32F103C8T6, X0 OPI-ZERO

Commit message: Updated design files
Parts:
- removed R40: 10K 1%, rcl:R-EU_R0603
- removed R41: 30K 1%, rcl:R-EU_R0603
- added R73, R74, R75: 10K, rcl:R-EU_R0603
- added UART2: (no value), pinhead:PINHD-1X3
- R12, R30: value 150K 1% -> 39K 1%
- R22, R23: value 390 -> 1K
- R34: value 30K 1% -> 10K 1%
- R49, R50, R51, R52, R53, R54, R55, R56, R57, R58, R59, R60, R61, R62, R63, R64, R66: value (none) -> 10K
- R5: value 51K 1% -> 10K 1%
- R6, R7: value 4.7K -> 3.3K
- R9: value (none) -> 120
Connections:
- removed net AD-VCC: R40.2, R41.1, U2.PB1
- removed net N$1: IC2.DE, X0.UART2_RTS/PA02
- removed net N$2: IC2.RO, X0.UART2_RX/PA01
- removed net N$9: IC2.DI, X0.UART2_TX/PA00
- new net U3DE: IC2.DE, IC2.RE/, R75.2, U2.PB2
- new net U3RX: IC2.RO, R74.2, U2.PB11
- new net U3TX: IC2.DI, R73.2, U2.PB10
- new net Z2RX: UART2.2, X0.UART2_RX/PA01
- new net Z2TX: UART2.1, X0.UART2_TX/PA00
- net GND: now also R75.1, UART2.3; no longer IC2.RE/, R40.1
- net VCC: now also C7.2, IC2.VCC, R73.1, R74.1; no longer R41.2
- net Z3V3: no longer C7.2, IC2.VCC
Other:
- moved on the sheet: I2C

Commit message: Update correct signal names
Parts:
- R15, R16, R18, R19, R21, R24, R26, R27, R32, R36, R38, R39, R43, R44, R46, R47: value (none) -> 220
- R17, R20, R25, R31, R37, R42, R45, R48: value (none) -> 100
- R65: value (none) -> 560
Other:
- moved on the sheet: R67
Changed lines of the file:
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@@
 <part name="OK7" library="optocoupler" deviceset="MOCD20*M" device="" technology="7"/>
 <part name="OK8" library="optocoupler" deviceset="MOCD20*M" device="" technology="7"/>
-<part name="R15" library="rcl" deviceset="R-EU_" device="R0603"/>
-<part name="R16" library="rcl" deviceset="R-EU_" device="R0603"/>
-<part name="R17" library="rcl" deviceset="R-EU_" device="R0603"/>
-<part name="R18" library="rcl" deviceset="R-EU_" device="R0603"/>
-<part name="R19" library="rcl" deviceset="R-EU_" device="R0603"/>
-<part name="R20" library="rcl" deviceset="R-EU_" device="R0603"/>
-<part name="R21" library="rcl" deviceset="R-EU_" device="R0603"/>
-<part name="R24" library="rcl" deviceset="R-EU_" device="R0603"/>
-<part name="R25" library="rcl" deviceset="R-EU_" device="R0603"/>
-<part name="R26" library="rcl" deviceset="R-EU_" device="R0603"/>
-<part name="R27" library="rcl" deviceset="R-EU_" device="R0603"/>
-<part name="R31" library="rcl" deviceset="R-EU_" device="R0603"/>
-<part name="R32" library="rcl" deviceset="R-EU_" device="R0603"/>
-<part name="R36" library="rcl" deviceset="R-EU_" device="R0603"/>
-<part name="R37" library="rcl" deviceset="R-EU_" device="R0603"/>
-<part name="R38" library="rcl" deviceset="R-EU_" device="R0603"/>
-<part name="R39" library="rcl" deviceset="R-EU_" device="R0603"/>
-<part name="R42" library="rcl" deviceset="R-EU_" device="R0603"/>
-<part name="R43" library="rcl" deviceset="R-EU_" device="R0603"/>
-<part name="R44" library="rcl" deviceset="R-EU_" device="R0603"/>
-<part name="R45" library="rcl" deviceset="R-EU_" device="R0603"/>
-<part name="R46" library="rcl" deviceset="R-EU_" device="R0603"/>
-<part name="R47" library="rcl" deviceset="R-EU_" device="R0603"/>
-<part name="R48" library="rcl" deviceset="R-EU_" device="R0603"/>
+<part name="R15" library="rcl" deviceset="R-EU_" device="R0603" value="220"/>
+<part name="R16" library="rcl" deviceset="R-EU_" device="R0603" value="220"/>
+<part name="R17" library="rcl" deviceset="R-EU_" device="R0603" value="100"/>
+<part name="R18" library="rcl" deviceset="R-EU_" device="R0603" value="220"/>
+<part name="R19" library="rcl" deviceset="R-EU_" device="R0603" value="220"/>
+<part name="R20" library="rcl" deviceset="R-EU_" device="R0603" value="100"/>
+<part name="R21" library="rcl" deviceset="R-EU_" device="R0603" value="220"/>
+<part name="R24" library="rcl" deviceset="R-EU_" device="R0603" value="220"/>
+<part name="R25" library="rcl" deviceset="R-EU_" device="R0603" value="100"/>
+<part name="R26" library="rcl" deviceset="R-EU_" device="R0603" value="220"/>
+<part name="R27" library="rcl" deviceset="R-EU_" device="R0603" value="220"/>
+<part name="R31" library="rcl" deviceset="R-EU_" device="R0603" value="100"/>
+<part name="R32" library="rcl" deviceset="R-EU_" device="R0603" value="220"/>
+<part name="R36" library="rcl" deviceset="R-EU_" device="R0603" value="220"/>
+<part name="R37" library="rcl" deviceset="R-EU_" device="R0603" value="100"/>
+<part name="R38" library="rcl" deviceset="R-EU_" device="R0603" value="220"/>
+<part name="R39" library="rcl" deviceset="R-EU_" device="R0603" value="220"/>
+<part name="R42" library="rcl" deviceset="R-EU_" device="R0603" value="100"/>
+<part name="R43" library="rcl" deviceset="R-EU_" device="R0603" value="220"/>
+<part name="R44" library="rcl" deviceset="R-EU_" device="R0603" value="220"/>
+<part name="R45" library="rcl" deviceset="R-EU_" device="R0603" value="100"/>
+<part name="R46" library="rcl" deviceset="R-EU_" device="R0603" value="220"/>
+<part name="R47" library="rcl" deviceset="R-EU_" device="R0603" value="220"/>
+<part name="R48" library="rcl" deviceset="R-EU_" device="R0603" value="100"/>
 <part name="R49" library="rcl" deviceset="R-EU_" device="R0603" value="10K"/>
 <part name="R50" library="rcl" deviceset="R-EU_" device="R0603" value="10K"/>
@@
 <part name="R64" library="rcl" deviceset="R-EU_" device="R0603" value="10K"/>
 <part name="OK9" library="optocoupler" deviceset="MOCD20*M" device="" technology="7"/>
-<part name="R65" library="rcl" deviceset="R-EU_" device="R0603"/>
+<part name="R65" library="rcl" deviceset="R-EU_" device="R0603" value="560"/>
 <part name="R66" library="rcl" deviceset="R-EU_" device="R0603" value="10K"/>
 <part name="C16" library="rcl" deviceset="C-EU" device="C1206" value="1.0"/>
@@
 <instance part="IC5" gate="G$1" x="-64.77" y="-52.07" rot="MR0"/>
 <instance part="Q1" gate="G$1" x="-185.42" y="-7.62" rot="MR0"/>
-<instance part="R67" gate="G$1" x="-162.56" y="-10.16"/>
+<instance part="R67" gate="G$1" x="-170.18" y="-10.16"/>
 <instance part="R68" gate="G$1" x="-162.56" y="-15.24"/>
 <instance part="C18" gate="G$1" x="-175.26" y="5.08" rot="R180"/>
@@
 <junction x="-132.08" y="68.58"/>
 <wire x1="-17.78" y1="-2.54" x2="-17.78" y2="2.54" width="0.1524" layer="91"/>
-<wire x1="-17.78" y1="2.54" x2="50.8" y2="2.54" width="0.1524" layer="91"/>
-<wire x1="50.8" y1="2.54" x2="50.8" y2="-7.62" width="0.1524" layer="91"/>
+<wire x1="-17.78" y1="2.54" x2="38.1" y2="2.54" width="0.1524" layer="91"/>
+<wire x1="38.1" y1="2.54" x2="38.1" y2="-7.62" width="0.1524" layer="91"/>
 <pinref part="R73" gate="G$1" pin="1"/>
 <wire x1="63.5" y1="-5.08" x2="63.5" y2="-7.62" width="0.1524" layer="91"/>
@@
 <wire x1="63.5" y1="-7.62" x2="76.2" y2="-7.62" width="0.1524" layer="91"/>
 <wire x1="76.2" y1="-7.62" x2="76.2" y2="-5.08" width="0.1524" layer="91"/>
-<wire x1="50.8" y1="-7.62" x2="63.5" y2="-7.62" width="0.1524" layer="91"/>
+<wire x1="38.1" y1="-7.62" x2="63.5" y2="-7.62" width="0.1524" layer="91"/>
 <junction x="-17.78" y="-2.54"/>
 <junction x="63.5" y="-7.62"/>
@@
 <pinref part="Q1" gate="G$1" pin="G"/>
 <pinref part="R67" gate="G$1" pin="1"/>
-<wire x1="-180.34" y1="-10.16" x2="-167.64" y2="-10.16" width="0.1524" layer="91"/>
+<wire x1="-180.34" y1="-10.16" x2="-175.26" y2="-10.16" width="0.1524" layer="91"/>
 </segment>
 </net>
@@
 <segment>
 <pinref part="R67" gate="G$1" pin="2"/>
-<wire x1="-157.48" y1="-10.16" x2="-154.94" y2="-10.16" width="0.1524" layer="91"/>
+<wire x1="-165.1" y1="-10.16" x2="-154.94" y2="-10.16" width="0.1524" layer="91"/>
 <wire x1="-154.94" y1="-10.16" x2="-154.94" y2="-15.24" width="0.1524" layer="91"/>
 <pinref part="R68" gate="G$1" pin="2"/>
