File: SmartNode/eagle/Make-v3.1/main-stm-03.1.brd (EAGLE design)
At the start: 131.8 x 67 mm, 152 parts, among them IC2 MAX3468CSA, IC4 78L33, IC5 MCP23017-E/SO-SOIC28, IC6 TPS56X200, IC7 LTC1694, Q1 IRLML2502, Q2 IRLML2502, U2 STM32F103C8T6, X0 OPI-ZERO

Commit message: Updated design files
Parts:
- removed R40: 10K 1%, rcl:R0603
- removed R41: 30K 1%, rcl:R0603
- added R73, R74, R75: 10K, rcl:R0603
- added UART2: (no value), pinhead:1X03
- moved C23 15.1 mm to (33.3, 18.4), flipped to the top, turned to 0 degrees
- moved R71 11.2 mm to (13.3, 45.1), flipped to the top, turned to 0 degrees
- moved R70 8.53 mm to (13.3, 43.2), flipped to the top, turned to 0 degrees
- moved Q2 4.26 mm to (18.4, 45.7), flipped to the top, turned to 270 degrees
Connections:
- removed net AD-VCC: R40.2, R41.1, U2.19
- removed net N$1: IC2.3, X0.22
- removed net N$2: IC2.1, X0.11
- removed net N$9: IC2.4, X0.13
- new net U3DE: IC2.2, IC2.3, R75.2, U2.20
- new net U3RX: IC2.1, R74.2, U2.22
- new net U3TX: IC2.4, R73.2, U2.21
- new net Z2RX: UART2.2, X0.11
- new net Z2TX: UART2.1, X0.13
- net GND: now also R75.1, UART2.3; no longer IC2.2, R40.1
- net VCC: now also C7.2, IC2.8, R73.1, R74.1; no longer R41.2
- net Z3V3: no longer C7.2, IC2.8
Routing:
- net N$1: track 47.4 -> 0.00 mm, vias 1 -> 0
- net N$9: track 32.5 -> 0.00 mm, vias 1 -> 0
- net U3TX: track 0.00 -> 32.2 mm, vias 0 -> 1
- net N$2: track 32.0 -> 0.00 mm, vias 1 -> 0
- net U3RX: track 0.00 -> 25.9 mm, vias 0 -> 1
- net U3DE: track 0.00 -> 24.6 mm, vias 0 -> 1
- net VCC: track 107.3 -> 130.2 mm
- net Z3V3: track 298.8 -> 278.2 mm
- net Z2TX: track 0.00 -> 13.5 mm
- net Z2RX: track 0.00 -> 13.5 mm
- net AD-VCC: track 6.64 -> 0.00 mm, vias 1 -> 0
- net GND: track 90.0 -> 86.4 mm, vias 77 -> 78
- net N$4: track 4.18 -> 7.47 mm, vias 0 -> 1
- net N$5: track 2.81 -> 4.29 mm
- net AD-3V3: track 12.1 -> 13.4 mm
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Other:
- board text added: "+ D C G"
- board text added: "H3.1"
- board text removed: "H2.2"
