File: SmartNode/eagle/Make-v3.1/main-stm-03.1.sch (EAGLE design)
At the start: 152 parts, among them IC2 MAX3468CSA, IC4 78L33, IC5 MCP23017-E/SO-SOIC28, IC6 TPS56X200, IC7 LTC1694, Q1 IRLML2502, Q2 IRLML2502, U2 STM32F103C8T6, X0 OPI-ZERO

Commit message: Updated design files
Parts:
- removed R40: 10K 1%, rcl:R-EU_R0603
- removed R41: 30K 1%, rcl:R-EU_R0603
- added R73, R74, R75: 10K, rcl:R-EU_R0603
- added UART2: (no value), pinhead:PINHD-1X3
Connections:
- removed net AD-VCC: R40.2, R41.1, U2.PB1
- removed net N$1: IC2.DE, X0.UART2_RTS/PA02
- removed net N$2: IC2.RO, X0.UART2_RX/PA01
- removed net N$9: IC2.DI, X0.UART2_TX/PA00
- new net U3DE: IC2.DE, IC2.RE/, R75.2, U2.PB2
- new net U3RX: IC2.RO, R74.2, U2.PB11
- new net U3TX: IC2.DI, R73.2, U2.PB10
- new net Z2RX: UART2.2, X0.UART2_RX/PA01
- new net Z2TX: UART2.1, X0.UART2_TX/PA00
- net GND: now also R75.1, UART2.3; no longer IC2.RE/, R40.1
- net VCC: now also C7.2, IC2.VCC, R73.1, R74.1; no longer R41.2
- net Z3V3: no longer C7.2, IC2.VCC
Other:
- moved on the sheet: I2C
